File: hardware/MultiRomCard.sch (KiCad schematic (older format))
At the start: 55 parts, among them P1 VC4000_Cartridge_Bus, P2 MicroSD_Breakout, P3 DISPLAY, P4 JUMPER1, P5 JUMPER2, P6 JUMPER3, P7 JUMPER4, SW1 UP, SW2 DOWN, SW3 SELECT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

Commit message: [PCB] New cap footprint with larger pads...
- ... should allow for easier hand soldering.
- Some minor reroutings to decrease copper loss when etching the board.
Parts:
- C1, C10, C11, C2, C3, C4, C5, C6, C7, C8, C9: footprint Capacitors_ThroughHole:C_Rect_L7_W2_P5 -> VC4000_MultiRom:C_Rect_L7_W2_P5_DIY
Changed lines of the file:
@@
 F 0 "C1" H 7025 6350 50  0000 L CNN
 F 1 ".1uF" H 7025 6150 50  0000 L CNN
-F 2 "Capacitors_ThroughHole:C_Rect_L7_W2_P5" H 7038 6100 30  0001 C CNN
+F 2 "VC4000_MultiRom:C_Rect_L7_W2_P5_DIY" H 7038 6100 30  0001 C CNN
 F 3 "" H 7000 6250 60  0000 C CNN
 	1    7000 6250
@@
 F 0 "C2" H 7325 6350 50  0000 L CNN
 F 1 ".1uF" H 7325 6150 50  0000 L CNN
-F 2 "Capacitors_ThroughHole:C_Rect_L7_W2_P5" H 7338 6100 30  0001 C CNN
+F 2 "VC4000_MultiRom:C_Rect_L7_W2_P5_DIY" H 7338 6100 30  0001 C CNN
 F 3 "" H 7300 6250 60  0000 C CNN
 	1    7300 6250
@@
 F 0 "C3" H 7625 6350 50  0000 L CNN
 F 1 ".1uF" H 7625 6150 50  0000 L CNN
-F 2 "Capacitors_ThroughHole:C_Rect_L7_W2_P5" H 7638 6100 30  0001 C CNN
+F 2 "VC4000_MultiRom:C_Rect_L7_W2_P5_DIY" H 7638 6100 30  0001 C CNN
 F 3 "" H 7600 6250 60  0000 C CNN
 	1    7600 6250
@@
 F 0 "C4" H 7925 6350 50  0000 L CNN
 F 1 ".1uF" H 7925 6150 50  0000 L CNN
-F 2 "Capacitors_ThroughHole:C_Rect_L7_W2_P5" H 7938 6100 30  0001 C CNN
+F 2 "VC4000_MultiRom:C_Rect_L7_W2_P5_DIY" H 7938 6100 30  0001 C CNN
 F 3 "" H 7900 6250 60  0000 C CNN
 	1    7900 6250
@@
 F 0 "C5" H 8225 6350 50  0000 L CNN
 F 1 ".1uF" H 8225 6150 50  0000 L CNN
-F 2 "Capacitors_ThroughHole:C_Rect_L7_W2_P5" H 8238 6100 30  0001 C CNN
+F 2 "VC4000_MultiRom:C_Rect_L7_W2_P5_DIY" H 8238 6100 30  0001 C CNN
 F 3 "" H 8200 6250 60  0000 C CNN
 	1    8200 6250
@@
 F 0 "C6" H 8525 6350 50  0000 L CNN
 F 1 ".1uF" H 8525 6150 50  0000 L CNN
-F 2 "Capacitors_ThroughHole:C_Rect_L7_W2_P5" H 8538 6100 30  0001 C CNN
+F 2 "VC4000_MultiRom:C_Rect_L7_W2_P5_DIY" H 8538 6100 30  0001 C CNN
 F 3 "" H 8500 6250 60  0000 C CNN
 	1    8500 6250
@@
 F 0 "C7" H 8825 6350 50  0000 L CNN
 F 1 ".1uF" H 8825 6150 50  0000 L CNN
-F 2 "Capacitors_ThroughHole:C_Rect_L7_W2_P5" H 8838 6100 30  0001 C CNN
+F 2 "VC4000_MultiRom:C_Rect_L7_W2_P5_DIY" H 8838 6100 30  0001 C CNN
 F 3 "" H 8800 6250 60  0000 C CNN
 	1    8800 6250
@@
 F 0 "C8" H 9125 6350 50  0000 L CNN
 F 1 ".1uF" H 9125 6150 50  0000 L CNN
-F 2 "Capacitors_ThroughHole:C_Rect_L7_W2_P5" H 9138 6100 30  0001 C CNN
+F 2 "VC4000_MultiRom:C_Rect_L7_W2_P5_DIY" H 9138 6100 30  0001 C CNN
 F 3 "" H 9100 6250 60  0000 C CNN
 	1    9100 6250
@@
 F 0 "C9" H 9425 6350 50  0000 L CNN
 F 1 ".1uF" H 9425 6150 50  0000 L CNN
-F 2 "Capacitors_ThroughHole:C_Rect_L7_W2_P5" H 9438 6100 30  0001 C CNN
+F 2 "VC4000_MultiRom:C_Rect_L7_W2_P5_DIY" H 9438 6100 30  0001 C CNN
 F 3 "" H 9400 6250 60  0000 C CNN
 	1    9400 6250
@@
 F 0 "C10" H 9725 6350 50  0000 L CNN
 F 1 ".1uF" H 9725 6150 50  0000 L CNN
-F 2 "Capacitors_ThroughHole:C_Rect_L7_W2_P5" H 9738 6100 30  0001 C CNN
+F 2 "VC4000_MultiRom:C_Rect_L7_W2_P5_DIY" H 9738 6100 30  0001 C CNN
 F 3 "" H 9700 6250 60  0000 C CNN
 	1    9700 6250
@@
 F 0 "C11" H 10025 6350 50  0000 L CNN
 F 1 ".1uF" H 10025 6150 50  0000 L CNN
-F 2 "Capacitors_ThroughHole:C_Rect_L7_W2_P5" H 10038 6100 30  0001 C CNN
+F 2 "VC4000_MultiRom:C_Rect_L7_W2_P5_DIY" H 10038 6100 30  0001 C CNN
 F 3 "" H 10000 6250 60  0000 C CNN
 	1    10000 6250
